File: templates/battery/default_18650_AP2112K.kicad_sch (KiCad schematic)
At the start: 6 parts

Commit message: update footprint related posotion in tp4056 and 18650 correct default_18650_AP2112K schematic
Parts:
- added BAT_R2: 810K, ErgoCai:R_0603, symbol Device:R_Small
- added BAT_R3: 2M, ErgoCai:R_0603, symbol Device:R_Small
Connections:
- net GND: now also BAT_R3.2
- net VBAT: now also BAT_R2.1
- new net BT_PIN: BAT_R2.2, BAT_R3.1

Commit message: update footprint lib to ergocai.pretty
Parts:
- BAT_D1: footprint ErgoCai:D_SOD-123 -> ErgoCai.pretty:D_SOD-123
- BAT_J1: footprint ErgoCai:Battery_Holder_18650_Nickel -> ErgoCai.pretty:Battery_Holder_18650_Nickel
- BAT_Q1: footprint ErgoCai:SOT-23 -> ErgoCai.pretty:SOT-23
- BAT_R1, BAT_R2, BAT_R3: footprint ErgoCai:R_0603 -> ErgoCai.pretty:R_0603
- BAT_SW1: footprint ErgoCai:MSK-12C02 -> ErgoCai.pretty:MSK-12C02
- BAT_U1: footprint Package_TO_SOT_SMD:SOT-23-5 -> ErgoCai.pretty:SOT-23-5
Changed lines of the file:
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@@
 			)
 		)
-		(property "Footprint" "ErgoCai:MSK-12C02"
+		(property "Footprint" "ErgoCai.pretty:MSK-12C02"
 			(at 94.615 69.85 0)
 			(effects
@@
 		)
 		(instances
-			(project "ergo_cai"
-				(path "/4ad52d44-7e09-4b14-9ca9-1745a5702ae6/4f209baf-4a6a-4aad-b42b-666d7fffdcd4"
+			(project ""
+				(path "/4ad52d44-7e09-4b14-9ca9-1745a5702ae6/559a5175-ec72-4734-ba4a-6993c402281d"
 					(reference "BAT_SW1")
 					(unit 1)
@@
 		)
 		(instances
-			(project "ergo_cai"
-				(path "/4ad52d44-7e09-4b14-9ca9-1745a5702ae6/4f209baf-4a6a-4aad-b42b-666d7fffdcd4"
+			(project ""
+				(path "/4ad52d44-7e09-4b14-9ca9-1745a5702ae6/559a5175-ec72-4734-ba4a-6993c402281d"
 					(reference "#PWR05")
 					(unit 1)
@@
 			)
 		)
-		(property "Footprint" "ErgoCai:R_0603"
+		(property "Footprint" "ErgoCai.pretty:R_0603"
 			(at 74.93 99.06 0)
 			(effects
@@
 		(pin "2"
 		)
-		(instances
-			(project "ergo_cai"
-				(path "/4ad52d44-7e09-4b14-9ca9-1745a5702ae6/4f209baf-4a6a-4aad-b42b-666d7fffdcd4"
-					(reference "BAT_R1")
-					(unit 1)
-				)
-			)
-		)
 	)
 	(symbol
@@
 			)
 		)
-		(property "Footprint" "ErgoCai:D_SOD-123"
+		(property "Footprint" "ErgoCai.pretty:D_SOD-123"
 			(at 81.28 93.98 90)
 			(effects
@@
 		(pin "2"
 		)
-		(instances
-			(project "ergo_cai"
-				(path "/4ad52d44-7e09-4b14-9ca9-1745a5702ae6/4f209baf-4a6a-4aad-b42b-666d7fffdcd4"
-					(reference "BAT_D1")
-					(unit 1)
-				)
-			)
-		)
 	)
 	(symbol
@@
 			)
 		)
-		(property "Footprint" "ErgoCai:SOT-23"
+		(property "Footprint" "ErgoCai.pretty:SOT-23"
 			(at 91.44 86.995 0)
 			(effects
@@
 		)
 		(instances
-			(project "ergo_cai"
-				(path "/4ad52d44-7e09-4b14-9ca9-1745a5702ae6/4f209baf-4a6a-4aad-b42b-666d7fffdcd4"
+			(project ""
+				(path "/4ad52d44-7e09-4b14-9ca9-1745a5702ae6/559a5175-ec72-4734-ba4a-6993c402281d"
 					(reference "BAT_Q1")
 					(unit 1)
@@
 			)
 		)
-		(property "Footprint" "Package_TO_SOT_SMD:SOT-23-5"
+		(property "Footprint" "ErgoCai.pretty:SOT-23-5"
 			(at 106.68 88.265 0)
 			(effects
@@
 		(instances
 			(project ""
-				(path "/4ad52d44-7e09-4b14-9ca9-1745a5702ae6/4f209baf-4a6a-4aad-b42b-666d7fffdcd4"
+				(path "/4ad52d44-7e09-4b14-9ca9-1745a5702ae6/559a5175-ec72-4734-ba4a-6993c402281d"
 					(reference "BAT_U1")
 					(unit 1)
@@
 		)
 		(instances
-			(project "ergo_cai"
-				(path "/4ad52d44-7e09-4b14-9ca9-1745a5702ae6/4f209baf-4a6a-4aad-b42b-666d7fffdcd4"
+			(project ""
+				(path "/4ad52d44-7e09-4b14-9ca9-1745a5702ae6/559a5175-ec72-4734-ba4a-6993c402281d"
 					(reference "#PWR012")
 					(unit 1)
@@
 			)
 		)
-		(property "Footprint" "ErgoCai:R_0603"
+		(property "Footprint" "ErgoCai.pretty:R_0603"
 			(at 125.73 50.8 0)
 			(effects
@@
 		(pin "2"
 		)
-		(instances
-			(project "ergo_cai"
-				(path "/4ad52d44-7e09-4b14-9ca9-1745a5702ae6/4f209baf-4a6a-4aad-b42b-666d7fffdcd4"
-					(reference "BAT_R2")
-					(unit 1)
-				)
-			)
-		)
 	)
 	(symbol
@@
 			)
 		)
-		(property "Footprint" "ErgoCai:Battery_Holder_18650_Nickel"
+		(property "Footprint" "ErgoCai.pretty:Battery_Holder_18650_Nickel"
 			(at 83.82 50.8 0)
 			(effects
@@
 		(pin "2"
 		)
-		(instances
-			(project "ergo_cai"
-				(path "/4ad52d44-7e09-4b14-9ca9-1745a5702ae6/4f209baf-4a6a-4aad-b42b-666d7fffdcd4"
-					(reference "BAT_J1")
-					(unit 1)
-				)
-			)
-		)
 	)
 	(symbol
@@
 		)
 		(instances
-			(project "ergo_cai"
-				(path "/4ad52d44-7e09-4b14-9ca9-1745a5702ae6/4f209baf-4a6a-4aad-b42b-666d7fffdcd4"
+			(project ""
+				(path "/4ad52d44-7e09-4b14-9ca9-1745a5702ae6/559a5175-ec72-4734-ba4a-6993c402281d"
 					(reference "#PWR04")
 					(unit 1)
@@
 			)
 		)
-		(property "Footprint" "ErgoCai:R_0603"
+		(property "Footprint" "ErgoCai.pretty:R_0603"
 			(at 135.89 50.8 0)
 			(effects
@@
 		(pin "2"
 		)
-		(instances
-			(project "ergo_cai"
-				(path "/4ad52d44-7e09-4b14-9ca9-1745a5702ae6/4f209baf-4a6a-4aad-b42b-666d7fffdcd4"
-					(reference "BAT_R3")
-					(unit 1)
-				)
-			)
-		)
 	)
 	(symbol
@@
 		)
 		(instances
-			(project "ergo_cai"
-				(path "/4ad52d44-7e09-4b14-9ca9-1745a5702ae6/4f209baf-4a6a-4aad-b42b-666d7fffdcd4"
+			(project ""
+				(path "/4ad52d44-7e09-4b14-9ca9-1745a5702ae6/559a5175-ec72-4734-ba4a-6993c402281d"
 					(reference "#PWR06")
 					(unit 1)
