File: templates/charging/default_TP4056.kicad_sch (KiCad schematic)
At the start: 6 parts

Commit message: update footprint lib to ergocai.pretty
Parts:
- CHRG_LED_CHRG1, CHRG_LED_STDBY1: footprint ErgoCai:LED_0603_1608Metric -> ErgoCai.pretty:LED_0603_1608Metric
- CHRG_R_CHRG1, CHRG_R_STDBY1: footprint ErgoCai:R_0603 -> ErgoCai.pretty:R_0603
- CHRG_U1: footprint Package_SO:SOIC-8-1EP_3.9x4.9mm_P1.27mm_EP2.29x3mm -> ErgoCai.pretty:SOIC-8-1EP_3.9x4.9mm_P1.27mm_EP2.29x3mm
Changed lines of the file:
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@@
 			)
 		)
-		(property "Footprint" "Package_SO:SOIC-8-1EP_3.9x4.9mm_P1.27mm_EP2.29x3mm"
+		(property "Footprint" "ErgoCai.pretty:SOIC-8-1EP_3.9x4.9mm_P1.27mm_EP2.29x3mm"
 			(at 83.82 63.5 0)
 			(effects
@@
 		)
 		(instances
-			(project "ergo_cai"
-				(path "/4ad52d44-7e09-4b14-9ca9-1745a5702ae6/250fc6fe-a9d9-4c83-8a52-c217220cf31a"
+			(project ""
+				(path "/4ad52d44-7e09-4b14-9ca9-1745a5702ae6/e8f99de7-8b9a-4508-9f90-208f83e7960a"
 					(reference "CHRG_U1")
 					(unit 1)
@@
 			)
 		)
-		(property "Footprint" "ErgoCai:R_0603"
+		(property "Footprint" "ErgoCai.pretty:R_0603"
 			(at 72.39 61.468 90)
 			(effects
@@
 		)
 		(instances
-			(project "ergo_cai"
-				(path "/4ad52d44-7e09-4b14-9ca9-1745a5702ae6/250fc6fe-a9d9-4c83-8a52-c217220cf31a"
+			(project ""
+				(path "/4ad52d44-7e09-4b14-9ca9-1745a5702ae6/e8f99de7-8b9a-4508-9f90-208f83e7960a"
 					(reference "CHRG_R_CHRG1")
 					(unit 1)
@@
 		)
 		(instances
-			(project "ergo_cai"
-				(path "/4ad52d44-7e09-4b14-9ca9-1745a5702ae6/250fc6fe-a9d9-4c83-8a52-c217220cf31a"
+			(project ""
+				(path "/4ad52d44-7e09-4b14-9ca9-1745a5702ae6/e8f99de7-8b9a-4508-9f90-208f83e7960a"
 					(reference "#PWR020")
 					(unit 1)
@@
 			)
 		)
-		(property "Footprint" "ErgoCai:R_0603"
+		(property "Footprint" "ErgoCai.pretty:R_0603"
 			(at 72.39 70.358 90)
 			(effects
@@
 		)
 		(instances
-			(project "ergo_cai"
-				(path "/4ad52d44-7e09-4b14-9ca9-1745a5702ae6/250fc6fe-a9d9-4c83-8a52-c217220cf31a"
+			(project ""
+				(path "/4ad52d44-7e09-4b14-9ca9-1745a5702ae6/e8f99de7-8b9a-4508-9f90-208f83e7960a"
 					(reference "CHRG_R_STDBY1")
 					(unit 1)
@@
 			)
 		)
-		(property "Footprint" "ErgoCai:LED_0603_1608Metric"
+		(property "Footprint" "ErgoCai.pretty:LED_0603_1608Metric"
 			(at 53.34 59.69 0)
 			(effects
@@
 		)
 		(instances
-			(project "ergo_cai"
-				(path "/4ad52d44-7e09-4b14-9ca9-1745a5702ae6/250fc6fe-a9d9-4c83-8a52-c217220cf31a"
+			(project ""
+				(path "/4ad52d44-7e09-4b14-9ca9-1745a5702ae6/e8f99de7-8b9a-4508-9f90-208f83e7960a"
 					(reference "CHRG_LED_CHRG1")
 					(unit 1)
@@
 			)
 		)
-		(property "Footprint" "ErgoCai:LED_0603_1608Metric"
+		(property "Footprint" "ErgoCai.pretty:LED_0603_1608Metric"
 			(at 53.34 68.58 0)
 			(effects
@@
 		)
 		(instances
-			(project "ergo_cai"
-				(path "/4ad52d44-7e09-4b14-9ca9-1745a5702ae6/250fc6fe-a9d9-4c83-8a52-c217220cf31a"
+			(project ""
+				(path "/4ad52d44-7e09-4b14-9ca9-1745a5702ae6/e8f99de7-8b9a-4508-9f90-208f83e7960a"
 					(reference "CHRG_LED_STDBY1")
 					(unit 1)
@@
 		(pin "2"
 		)
-		(instances
-			(project "ergo_cai"
-				(path "/4ad52d44-7e09-4b14-9ca9-1745a5702ae6/250fc6fe-a9d9-4c83-8a52-c217220cf31a"
-					(reference "CHRG_R_PROG1")
-					(unit 1)
-				)
-			)
-		)
-	)
+	)
