File: templates/mcu/nRF52840_holyiot_18010.kicad_sch (KiCad schematic)
At the start: 3 parts

Commit message: correct reset button path
Parts:
- MCU_SW1: footprint ErgoCai:K2-1187SQ -> ErgoCai.pretty:K2-1187SQ
Changed lines of the file:
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@@
 			)
 		)
-		(property "Footprint" "ErgoCai:K2-1187SQ"
+		(property "Footprint" "ErgoCai.pretty:K2-1187SQ"
 			(at 134.62 38.1 0)
 			(effects
