File: e-paper/1.02inch-socket-right/1.02inch-socket-right.kicad_sch (KiCad schematic)
At the start: 2 parts

Commit message: update e-papert
Parts:
- added EPM_AREA1: MountingHole, ErgoCai.pretty:e-paper_1.02inch_area, symbol Mechanical:MountingHole
- added EPM_GAP1: MountingHole, ErgoCai.pretty:e-paper_1.02inch_gap, symbol Mechanical:MountingHole
- added EPM_H2, EPM_H3, EPM_H4: MountingHole, ErgoCai.pretty:MountingHole_2.2mm_M2_DIN965, symbol Mechanical:MountingHole
- EPM_H1: footprint ErgoCai.pretty:e-paper_1.02inch_mount -> ErgoCai.pretty:MountingHole_2.2mm_M2_DIN965
